Commit message: Added RAL 7016 to common_materials

File: kuka_resources/urdf/common_materials.xacro (robot description, xacro)
@@ -152,3 +152,8 @@
     </material>
   </xacro:macro>
+  <xacro:macro name="material_kuka_anthracite_gray">
+    <material name="">
+      <color rgba="${colour_kuka_anthracite_gray}"/>
+    </material>
+  </xacro:macro>
 </robot>
