Commit message: Gazebo fixes

File: kuka_kr10_gazebo/urdf/kr10.xacro (robot description, xacro)
@@ -1,5 +1,5 @@
 <?xml version="1.0" ?>
 <robot name="kuka_kr10_gazebo" xmlns:xacro="http://ros.org/wiki/xacro">
-  <!-- TX90 -->
+  <!-- kr10 -->
   <xacro:include filename="$(find kuka_kr10_gazebo)/urdf/kr10_macro.xacro"/>
   <xacro:kuka_kr10_robot prefix=""/>

File: kuka_kr10_gazebo/urdf/kr10_macro.xacro (robot description, xacro)
@@ -69,25 +69,25 @@
   <!-- Gazebo-specific link properties -->
   <gazebo reference="${prefix}base_link">
-    <material>Gazebo/Yellow</material>
+    <material>Gazebo/Black</material>
     <turnGravityOff>true</turnGravityOff>
   </gazebo>
   <gazebo reference="${prefix}link_1">
-    <material>Gazebo/Yellow</material>
+    <material>Gazebo/DarkGrey</material>
     <turnGravityOff>true</turnGravityOff>
   </gazebo>
   <gazebo reference="${prefix}link_2">
-    <material>Gazebo/Yellow</material>
+    <material>Gazebo/DarkGrey</material>
     <turnGravityOff>true</turnGravityOff>
   </gazebo>
   <gazebo reference="${prefix}link_3">
-    <material>Gazebo/Yellow</material>
+    <material>Gazebo/DarkGrey</material>
     <turnGravityOff>true</turnGravityOff>
   </gazebo>
   <gazebo reference="${prefix}link_4">
-    <material>Gazebo/Yellow</material>
+    <material>Gazebo/DarkGrey</material>
     <turnGravityOff>true</turnGravityOff>
   </gazebo>
   <gazebo reference="${prefix}link_5">
-    <material>Gazebo/Grey</material>
+    <material>Gazebo/DarkGrey</material>
     <turnGravityOff>true</turnGravityOff>
   </gazebo>
