Commit message: Joint name fices

File: kuka_kr10_gazebo/urdf/kr10_macro.xacro (robot description, xacro)
@@ -9,6 +9,6 @@
     <robotNamespace>/${prefix}</robotNamespace>
     <type>transmission_interface/SimpleTransmission</type>
-    <joint name="${prefix}joint_1">
-      <hardwareInterface>PositionJointInterface</hardwareInterface>
+    <joint name="${prefix}joint_a1">
+      <hardwareInterface>hardware_interface/PositionJointInterface</hardwareInterface>
     </joint>
     <actuator name="${prefix}motor1">
@@ -19,6 +19,6 @@
     <robotNamespace>/${prefix}</robotNamespace>
     <type>transmission_interface/SimpleTransmission</type>
-    <joint name="${prefix}joint_2">
-      <hardwareInterface>PositionJointInterface</hardwareInterface>
+    <joint name="${prefix}joint_a2">
+      <hardwareInterface>hardware_interface/PositionJointInterface</hardwareInterface>
     </joint>
     <actuator name="${prefix}motor2">
@@ -29,6 +29,6 @@
     <robotNamespace>/${prefix}</robotNamespace>
     <type>transmission_interface/SimpleTransmission</type>
-    <joint name="${prefix}joint_3">
-      <hardwareInterface>PositionJointInterface</hardwareInterface>
+    <joint name="${prefix}joint_a3">
+      <hardwareInterface>hardware_interface/PositionJointInterface</hardwareInterface>
     </joint>
     <actuator name="${prefix}motor3">
@@ -39,6 +39,6 @@
     <robotNamespace>/${prefix}</robotNamespace>
     <type>transmission_interface/SimpleTransmission</type>
-    <joint name="${prefix}joint_4">
-      <hardwareInterface>PositionJointInterface</hardwareInterface>
+    <joint name="${prefix}joint_a4">
+      <hardwareInterface>hardware_interface/PositionJointInterface</hardwareInterface>
     </joint>
     <actuator name="${prefix}motor4">
@@ -49,6 +49,6 @@
     <robotNamespace>/${prefix}</robotNamespace>
     <type>transmission_interface/SimpleTransmission</type>
-    <joint name="${prefix}joint_5">
-      <hardwareInterface>PositionJointInterface</hardwareInterface>
+    <joint name="${prefix}joint_a5">
+      <hardwareInterface>hardware_interface/PositionJointInterface</hardwareInterface>
     </joint>
     <actuator name="${prefix}motor5">
@@ -59,6 +59,6 @@
     <robotNamespace>/${prefix}</robotNamespace>
     <type>transmission_interface/SimpleTransmission</type>
-    <joint name="${prefix}joint_6">
-      <hardwareInterface>PositionJointInterface</hardwareInterface>
+    <joint name="${prefix}joint_a6">
+      <hardwareInterface>hardware_interface/PositionJointInterface</hardwareInterface>
     </joint>
     <actuator name="${prefix}motor6">

Commit message: Minor changes

File: kuka_kr10_gazebo/urdf/kr10_macro.xacro (robot description, xacro)
@@ -73,5 +73,4 @@
   </gazebo>
   <gazebo reference="${prefix}link_1">
-<<<<<<< HEAD
     <material>Gazebo/DarkGrey</material>
     <turnGravityOff>true</turnGravityOff>
@@ -91,23 +90,4 @@
   <gazebo reference="${prefix}link_5">
     <material>Gazebo/DarkGrey</material>
-=======
-    <material>Gazebo/Orange</material>
-    <turnGravityOff>true</turnGravityOff>
-  </gazebo>
-  <gazebo reference="${prefix}link_2">
-    <material>Gazebo/Orange</material>
-    <turnGravityOff>true</turnGravityOff>
-  </gazebo>
-  <gazebo reference="${prefix}link_3">
-    <material>Gazebo/Orange</material>
-    <turnGravityOff>true</turnGravityOff>
-  </gazebo>
-  <gazebo reference="${prefix}link_4">
-    <material>Gazebo/Orange</material>
-    <turnGravityOff>true</turnGravityOff>
-  </gazebo>
-  <gazebo reference="${prefix}link_5">
-    <material>Gazebo/Orange</material>
->>>>>>> b1bbeb3c961b0bfd8cc234cdedf3a63034f573c1
     <turnGravityOff>true</turnGravityOff>
   </gazebo>
