Commit message: Incorporated new meshes w/o errors by bretthemes

File: kuka_kr10_support/urdf/kr10r1100sixx_macro.xacro (robot description, xacro)
@@ -1,4 +1,4 @@
 <?xml version="1.0"?>
-<robot xmlns:xacro="http://ros.org/wiki/xacro">
+<robot xmlns:xacro="http://wiki.ros.org/xacro">
   <xacro:include filename="$(find kuka_resources)/urdf/common_constants.xacro"/>
   <xacro:include filename="$(find kuka_resources)/urdf/common_materials.xacro"/>
@@ -8,7 +8,7 @@
         <origin xyz="0 0 0" rpy="0 0 0"/>
         <geometry>
-          <mesh filename="package://kuka_kr10_support/meshes/kr10r1100sixx/visual/base.stl" />
+          <mesh filename="package://kuka_kr10_support/meshes/kr10r1100sixx/visual/base.dae" />
         </geometry>
- 	      <xacro:material_kuka_black />
+        <xacro:material_kuka_black />
       </visual>
       <collision>
@@ -23,5 +23,5 @@
         <origin xyz="0 0 0" rpy="0 0 0"/>
         <geometry>
-          <mesh filename="package://kuka_kr10_support/meshes/kr10r1100sixx/visual/link_1.stl" />
+          <mesh filename="package://kuka_kr10_support/meshes/kr10r1100sixx/collision/link_1.stl" />
         </geometry>
         <xacro:material_kuka_anthracite_gray />
@@ -38,5 +38,5 @@
         <origin xyz="0 0 0" rpy="0 0 0"/>
         <geometry>
-          <mesh filename="package://kuka_kr10_support/meshes/kr10r1100sixx/visual/link_2.stl"/>
+          <mesh filename="package://kuka_kr10_support/meshes/kr10r1100sixx/collision/link_2.stl"/>
         </geometry>
         <xacro:material_kuka_anthracite_gray />
@@ -53,5 +53,5 @@
         <origin xyz="0 0 0" rpy="0 0 0"/>
         <geometry>
-          <mesh filename="package://kuka_kr10_support/meshes/kr10r1100sixx/visual/link_3.stl" />
+          <mesh filename="package://kuka_kr10_support/meshes/kr10r1100sixx/collision/link_3.stl" />
         </geometry>
         <xacro:material_kuka_anthracite_gray />
@@ -68,5 +68,5 @@
         <origin xyz="0 0 0" rpy="0 0 0"/>
         <geometry>
-          <mesh filename="package://kuka_kr10_support/meshes/kr10r1100sixx/visual/link_4.stl" />
+          <mesh filename="package://kuka_kr10_support/meshes/kr10r1100sixx/collision/link_4.stl" />
         </geometry>
         <xacro:material_kuka_anthracite_gray />
@@ -83,5 +83,5 @@
         <origin xyz="0 0 0" rpy="0 0 0"/>
         <geometry>
-          <mesh filename="package://kuka_kr10_support/meshes/kr10r1100sixx/visual/link_5.stl" />
+          <mesh filename="package://kuka_kr10_support/meshes/kr10r1100sixx/collision/link_5.stl" />
         </geometry>
         <xacro:material_kuka_anthracite_gray />
@@ -98,5 +98,5 @@
         <origin xyz="0 0 0" rpy="0 0 0"/>
         <geometry>
-          <mesh filename="package://kuka_kr10_support/meshes/kr10r1100sixx/visual/link_6.stl" />
+          <mesh filename="package://kuka_kr10_support/meshes/kr10r1100sixx/collision/link_6.stl" />
         </geometry>
         <xacro:material_kuka_pedestal />

Commit message: Cherry-pick merge visual holes

File: kuka_kr10_support/urdf/kr10r1100sixx_macro.xacro (robot description, xacro)
@@ -8,5 +8,5 @@
         <origin xyz="0 0 0" rpy="0 0 0"/>
         <geometry>
-          <mesh filename="package://kuka_kr10_support/meshes/kr10r1100sixx/visual/base.dae" />
+          <mesh filename="package://kuka_kr10_support/meshes/kr10r1100sixx/visual/base_link.stl" />
         </geometry>
         <xacro:material_kuka_black />
@@ -15,5 +15,5 @@
         <origin xyz="0 0 0" rpy="0 0 0"/>
         <geometry>
-          <mesh filename="package://kuka_kr10_support/meshes/kr10r1100sixx/collision/base.stl" />
+          <mesh filename="package://kuka_kr10_support/meshes/kr10r1100sixx/collision/base_link.stl" />
         </geometry>
       </collision>

Commit message: Added artificial joint limits to prevent weird movements

File: kuka_kr10_support/urdf/kr10r1100sixx_macro.xacro (robot description, xacro)
@@ -183,5 +183,6 @@
       <child link="${prefix}link_4"/>
       <axis xyz="-1 0 0"/>
-      <limit effort="0" lower="${-DEG2RAD * 185}" upper="${DEG2RAD * 185}" velocity="${DEG2RAD * 381}"/>
+      <!-- limit effort="0" lower="${-DEG2RAD * 185}" upper="${DEG2RAD * 185}" velocity="${DEG2RAD * 381}"/ -->
+      <limit effort="0" lower="${-DEG2RAD * 90}" upper="${DEG2RAD * 90}" velocity="${DEG2RAD * 381}"/>
     </joint>
     <joint name="${prefix}joint_a5" type="revolute">
@@ -197,5 +198,6 @@
       <child link="${prefix}link_6"/>
       <axis xyz="-1 0 0"/>
-      <limit effort="0" lower="${-DEG2RAD * 350}" upper="${DEG2RAD * 350}" velocity="${DEG2RAD * 615}"/>
+      <!-- limit effort="0" lower="${-DEG2RAD * 350}" upper="${DEG2RAD * 350}" velocity="${DEG2RAD * 615}"/ -->
+      <limit effort="0" lower="${-DEG2RAD * 180}" upper="${DEG2RAD * 180}" velocity="${DEG2RAD * 615}"/>
     </joint>
     <joint name="${prefix}joint_a6-tool0" type="fixed">
